Commit message: update the sensor plugin in robot model

File: zjlrobotone/urdf/zjlrobotone.urdf (robot description, URDF)
Before this commit: robot zjlrobotone, 26 links, 25 joints
Links:
- removed link gsensor
- removed link gyrometer
- removed link lfsensor
- removed link rfsensor
- added link left_foot_earth_link, mass 0.1; collision box size=0.3 0.2 0.03; visual box size=0.3 0.2 0.03
- added link right_foot_earth_link, mass 0.1; collision box size=0.3 0.2 0.03; visual box size=0.3 0.2 0.03
Joints:
- removed joint gsensor_JOINT
- removed joint gyrometer_JOINT
- removed joint lfsensor_JOINT
- removed joint rfsensor_JOINT
- added joint left_foot_earth: type revolute, parent left_foot_Link, child left_foot_earth_link, origin xyz=0 0 0 rpy=0 0 0, axis 0 1 0, limit lower=-0 upper=0 effort=100 velocity=100
- added joint right_foot_earth: type revolute, parent right_foot_Link, child right_foot_earth_link, origin xyz=0 0 0 rpy=0 0 0, axis 0 1 0, limit lower=-0 upper=0 effort=100 velocity=100
- joint left_ankle_pitch: origin xyz=0 0 0 rpy=0 0 0 -> xyz=0 0 0 rpy=0 -0.149307 0
- joint left_ankle_roll: axis -1 0 0 -> 1 0 0
- joint left_elbow_pitch: axis 0 -1 0 -> 0 1 0
- joint left_hip_pitch: origin xyz=0 0 0 rpy=0 0 0 -> xyz=0 0 0 rpy=0 -0.107303 0
- joint left_hip_roll: axis -1 0 0 -> 1 0 0
- joint left_hip_yaw: axis 0 0 -1 -> 0 0 1
- joint left_knee_pitch: origin xyz=0 0.013000000000026 -0.29999999999994 rpy=0 0 0 -> xyz=0 0.013000000000026 -0.29999999999994 rpy=0 0.257133 0
- joint left_shoulder_pitch: axis 0 -1 0 -> 0 1 0
- joint left_shoulder_roll: axis -1 0 0 -> 1 0 0
- joint neck_yaw: axis 0 0 -1 -> 0 0 1
- joint right_ankle_pitch: origin xyz=0 0 0 rpy=0 0 0 -> xyz=0 0 0 rpy=0 -0.149307 0
- joint right_ankle_roll: axis -1 0 0 -> 1 0 0
- joint right_hip_pitch: origin xyz=0 0 0 rpy=0 0 0 -> xyz=0 0 0 rpy=0 -0.107303 0
- joint right_hip_roll: axis -1 0 0 -> 1 0 0
- joint right_hip_yaw: axis 0 0 -1 -> 0 0 1
- joint right_knee_pitch: origin xyz=0 -0.0119999999999984 -0.3 rpy=0 0 0 -> xyz=0 -0.0119999999999984 -0.3 rpy=0 0.257133 0
- joint right_shoulder_roll: axis -1 0 0 -> 1 0 0
- joint trunk_link-base_fixed_joint: origin xyz=0 0 0 rpy=0 0 0 -> xyz=0 0 0.02 rpy=0 0 0
